Commit message: refactor: add inertia

File: ex01/cat_urdf_robot/urdf/robot.urdf (robot description, URDF)
Before this commit: robot myfirst, 14 links, 13 joints
Links:
- link back_left_leg: mass None -> 0.5
- link back_left_wheel: mass None -> 0.1
- link back_right_leg: mass None -> 0.5
- link back_right_wheel: mass None -> 0.1
- link base_link: mass None -> 3
- link front_left_leg: mass None -> 0.5
- link front_left_wheel: mass None -> 0.1
- link front_right_leg: mass None -> 0.5
- link front_right_wheel: mass None -> 0.1
- link head: mass None -> 1
- link neck: mass None -> 0.05
- link tail: mass None -> 0.1
